File: Source Files/PCB/BBQino/Arduino.sch (KiCad schematic (older format))
At the start: 1 part

Commit message: relay footprint
Parts:
- A?: symbol MCU_Module:Arduino_UNO_R3 -> BBQino-rescue:Arduino_UNO_R3-MCU_Module
Changed lines of the file:
@@
 $EndDescr
 $Comp
-L MCU_Module:Arduino_UNO_R3 A?
+L BBQino-rescue:Arduino_UNO_R3-MCU_Module A?
 U 1 1 613FC931
 P 2900 3200
@@
 $EndComp
 $Comp
-L power:GNDD #PWR?
+L BBQino-rescue:GNDD-power #PWR?
 U 1 1 6143AD0C
 P 3000 4400
