File: Source Files/PCB/BBQino/Power.sch (KiCad schematic (older format))
At the start: 9 parts, among them Q1 IPD068P03L3G

Commit message: relay footprint
Parts:
- C? (x4): symbol Device:C -> BBQino-rescue:C-Device
- DZ1: symbol Device:D_Zener_ALT -> BBQino-rescue:D_Zener_ALT-Device
- J?: symbol Connector:Screw_Terminal_01x02 -> BBQino-rescue:Screw_Terminal_01x02-Connector
- Q1: symbol Device:Q_PMOS_GDS -> BBQino-rescue:Q_PMOS_GDS-Device
- R1: symbol Device:R_US -> BBQino-rescue:R_US-Device
- U?: symbol Regulator_Linear:ADP7142ARDZ-5.0 -> BBQino-rescue:ADP7142ARDZ-5.0-Regulator_Linear
Changed lines of the file:
@@
 $EndDescr
 $Comp
-L Connector:Screw_Terminal_01x02 J?
+L BBQino-rescue:Screw_Terminal_01x02-Connector J?
 U 1 1 6143D9E7
 P 1250 1250
@@
 $EndComp
 $Comp
-L Device:D_Zener_ALT DZ1
+L BBQino-rescue:D_Zener_ALT-Device DZ1
 U 1 1 61441178
 P 2500 1350
@@
 $EndComp
 $Comp
-L Device:R_US R1
+L BBQino-rescue:R_US-Device R1
 U 1 1 61441EC4
 P 2100 1700
@@
 $EndComp
 $Comp
-L Device:C C?
+L BBQino-rescue:C-Device C?
 U 1 1 61442C4C
 P 2500 1700
@@
 	1450 1150 1900 1150
 $Comp
-L power:+12V #PWR?
+L BBQino-rescue:+12V-power #PWR?
 U 1 1 6144570A
 P 2500 1150
@@
 Connection ~ 2500 1150
 $Comp
-L power:GNDPWR #PWR?
+L BBQino-rescue:GNDPWR-power #PWR?
 U 1 1 61445C4C
 P 2500 1850
@@
 Connection ~ 2500 1850
 $Comp
-L Device:Q_PMOS_GDS Q1
+L BBQino-rescue:Q_PMOS_GDS-Device Q1
 U 1 1 614469CB
 P 2100 1250
@@
 Analog 5V POWER RAIL\n
 $Comp
-L Device:C C?
+L BBQino-rescue:C-Device C?
 U 1 1 6144ECB3
 P 3250 3250
@@
 $EndComp
 $Comp
-L Device:C C?
+L BBQino-rescue:C-Device C?
 U 1 1 6144F727
 P 1650 3350
@@
 $EndComp
 $Comp
-L power:+12V #PWR?
+L BBQino-rescue:+12V-power #PWR?
 U 1 1 614537EF
 P 1650 3050
@@
 	3100 3100 2850 3100
 $Comp
-L power:+5VA #PWR?
+L BBQino-rescue:+5VA-power #PWR?
 U 1 1 61456D2F
 P 3100 3050
@@
 $EndComp
 $Comp
-L power:GNDA #PWR?
+L BBQino-rescue:GNDA-power #PWR?
 U 1 1 61457278
 P 3250 3600
@@
 $EndComp
 $Comp
-L power:GNDPWR #PWR?
+L BBQino-rescue:GNDPWR-power #PWR?
 U 1 1 61459FC8
 P 2450 3650
@@
 	3100 3100 3100 3050
 $Comp
-L Regulator_Linear:ADP7142ARDZ-5.0 U?
+L BBQino-rescue:ADP7142ARDZ-5.0-Regulator_Linear U?
 U 1 1 614681CA
 P 2450 3200
@@
 	3100 3100 3250 3100
 $Comp
-L Device:C C?
+L BBQino-rescue:C-Device C?
 U 1 1 61474DD5
 P 2900 3500
@@
 	2900 3700 2900 3650
 $Comp
-L power:GNDA #PWR?
+L BBQino-rescue:GNDA-power #PWR?
 U 1 1 61476818
 P 2900 3700
