File: Source Files/PCB/BBQino/boardUtils.sch (KiCad schematic (older format))
At the start: 6 parts, among them U99 24LC512

Commit message: relay footprint
Parts:
- C?: symbol Device:C -> BBQino-rescue:C-Device
- EN_W: symbol Jumper:Jumper_3_Bridged12 -> BBQino-rescue:Jumper_3_Bridged12-Jumper
- J_A0, J_A1, J_A2: symbol Connector:Conn_01x03_Male -> BBQino-rescue:Conn_01x03_Male-Connector
- U99: symbol Memory_EEPROM:24LC512 -> BBQino-rescue:24LC512-Memory_EEPROM
Changed lines of the file:
@@
 $EndDescr
 $Comp
-L Memory_EEPROM:24LC512 U99
+L BBQino-rescue:24LC512-Memory_EEPROM U99
 U 1 1 6139200A
 P 2800 2100
@@
 $EndComp
 $Comp
-L Connector:Conn_01x03_Male J_A0
+L BBQino-rescue:Conn_01x03_Male-Connector J_A0
 U 1 1 61396B54
 P 1500 2600
@@
 	2800 1350 2800 1500
 $Comp
-L Connector:Conn_01x03_Male J_A1
+L BBQino-rescue:Conn_01x03_Male-Connector J_A1
 U 1 1 613A016A
 P 1500 3050
@@
 $EndComp
 $Comp
-L Connector:Conn_01x03_Male J_A2
+L BBQino-rescue:Conn_01x03_Male-Connector J_A2
 U 1 1 613A06AE
 P 1500 3550
@@
 EEPROM ADDRESS
 $Comp
-L Device:C C?
+L BBQino-rescue:C-Device C?
 U 1 1 613A7946
 P 4100 1700
@@
 	4100 1500 4100 1550
 $Comp
-L power:GNDD #PWR?
+L BBQino-rescue:GNDD-power #PWR?
 U 1 1 613AC7D9
 P 4100 1850
@@
 $EndComp
 $Comp
-L power:GNDD #PWR?
+L BBQino-rescue:GNDD-power #PWR?
 U 1 1 613B1156
 P 2800 2900
@@
 $EndComp
 $Comp
-L power:+5VD #PWR?
+L BBQino-rescue:+5VD-power #PWR?
 U 1 1 613B25A5
 P 2800 1350
@@
 $EndComp
 $Comp
-L Jumper:Jumper_3_Bridged12 EN_W
+L BBQino-rescue:Jumper_3_Bridged12-Jumper EN_W
 U 1 1 613B5C58
 P 3650 2500
@@
 	3500 2200 3500 2500
 $Comp
-L power:+5VD #PWR?
+L BBQino-rescue:+5VD-power #PWR?
 U 1 1 613B886B
 P 3650 2250
@@
 $EndComp
 $Comp
-L power:GNDD #PWR?
+L BBQino-rescue:GNDD-power #PWR?
 U 1 1 613BA173
 P 3650 2750
