File: Source Files/PCB/BBQino/boardUtils.sch (KiCad schematic (older format))
At the start: 6 parts, among them U99 24LC512

Commit message: 230V section first Draft. Added external module on top of the shield for the 230V section
Parts:
- gave numbers to parts that had none: 1
- renumbered EN_W to EN_W1
Changed lines of the file:
@@
 EEPROM ADDRESS
 $Comp
-L BBQino-rescue:C-Device C?
+L BBQino-rescue:C-Device C1
 U 1 1 613A7946
 P 4100 1700
-F 0 "C?" H 4215 1746 50  0000 L CNN
+F 0 "C1" H 4215 1746 50  0000 L CNN
 F 1 "C" H 4215 1655 50  0000 L CNN
 F 2 "" H 4138 1550 50  0001 C CNN
@@
 	4100 1500 4100 1550
 $Comp
-L BBQino-rescue:GNDD-power #PWR?
+L BBQino-rescue:GNDD-power #PWR0101
 U 1 1 613AC7D9
 P 4100 1850
-F 0 "#PWR?" H 4100 1600 50  0001 C CNN
+F 0 "#PWR0101" H 4100 1600 50  0001 C CNN
 F 1 "GNDD" H 4104 1695 50  0000 C CNN
 F 2 "" H 4100 1850 50  0001 C CNN
@@
 $EndComp
 $Comp
-L BBQino-rescue:GNDD-power #PWR?
+L BBQino-rescue:GNDD-power #PWR0102
 U 1 1 613B1156
 P 2800 2900
-F 0 "#PWR?" H 2800 2650 50  0001 C CNN
+F 0 "#PWR0102" H 2800 2650 50  0001 C CNN
 F 1 "GNDD" H 2804 2745 50  0000 C CNN
 F 2 "" H 2800 2900 50  0001 C CNN
@@
 $EndComp
 $Comp
-L BBQino-rescue:+5VD-power #PWR?
+L BBQino-rescue:+5VD-power #PWR0103
 U 1 1 613B25A5
 P 2800 1350
-F 0 "#PWR?" H 2800 1200 50  0001 C CNN
+F 0 "#PWR0103" H 2800 1200 50  0001 C CNN
 F 1 "+5VD" H 2815 1523 50  0000 C CNN
 F 2 "" H 2800 1350 50  0001 C CNN
@@
 $EndComp
 $Comp
-L BBQino-rescue:Jumper_3_Bridged12-Jumper EN_W
+L BBQino-rescue:Jumper_3_Bridged12-Jumper EN_W1
 U 1 1 613B5C58
 P 3650 2500
-F 0 "EN_W" V 3650 2567 50  0000 L CNN
+F 0 "EN_W1" V 3650 2567 50  0000 L CNN
 F 1 "Jumper_3_Bridged12" V 3695 2567 50  0001 L CNN
 F 2 "Jumper:SolderJumper-3_P1.3mm_Open_Pad1.0x1.5mm_NumberLabels" H 3650 2500 50  0001 C CNN
@@
 	3500 2200 3500 2500
 $Comp
-L BBQino-rescue:+5VD-power #PWR?
+L BBQino-rescue:+5VD-power #PWR0104
 U 1 1 613B886B
 P 3650 2250
-F 0 "#PWR?" H 3650 2100 50  0001 C CNN
+F 0 "#PWR0104" H 3650 2100 50  0001 C CNN
 F 1 "+5VD" H 3665 2423 50  0000 C CNN
 F 2 "" H 3650 2250 50  0001 C CNN
@@
 $EndComp
 $Comp
-L BBQino-rescue:GNDD-power #PWR?
+L BBQino-rescue:GNDD-power #PWR0105
 U 1 1 613BA173
 P 3650 2750
-F 0 "#PWR?" H 3650 2500 50  0001 C CNN
+F 0 "#PWR0105" H 3650 2500 50  0001 C CNN
 F 1 "GNDD" H 3654 2595 50  0000 C CNN
 F 2 "" H 3650 2750 50  0001 C CNN
