File: Source Files/PCB/BBQino/_autosave-BBQino.kicad_pcb (KiCad board)
At the start: 2 copper layers, 113 x 53.3 mm, 29 parts, among them J1 VIN < 13V, J2 230V input, J3 230V out, K1 FTR-MYAA005D, K2 FTR-MYAA005D, Q1 IPD068P03L3G, U1 ADP7142ARDZ-5.0, U99 24LC512

Commit message: added current sense on motor side
Parts:
- added C2: 2.2uF, Capacitor_SMD:C_0805_2012Metric_Pad1.18x1.45mm_HandSolder, F.Cu at (55.9, 111.5)
- added C3: 10nF, Capacitor_SMD:C_0805_2012Metric_Pad1.18x1.45mm_HandSolder, F.Cu at (60.7, 111.5)
- added C4: 1nF, Capacitor_SMD:C_0805_2012Metric_Pad1.18x1.45mm_HandSolder, F.Cu at (80.2, 101.9)
- added C5: 2.2uF, Capacitor_SMD:C_0805_2012Metric_Pad1.18x1.45mm_HandSolder, F.Cu at (65.5, 111.5)
- added IC2: DG4052EEN-T1-GE4, BBQino:QFN40P180X260X60-16N-D, F.Cu at (104.2, 96.4)
- added IC3: MAX6675ISA+T, BBQino:SOIC127P600X175-8N, F.Cu at (97.9, 97.2)
- added Q2: DMP4051LK3, Package_TO_SOT_SMD:TO-252-3_TabPin2, F.Cu at (59.5, 97.9)
- added Q3: DMN4040SK3, Package_TO_SOT_SMD:TO-252-3_TabPin2, F.Cu at (59.5, 106.0)
- added Q4: DMP4051LK3, Package_TO_SOT_SMD:TO-252-3_TabPin2, F.Cu at (71.7, 97.9)
- added Q5: DMN4040SK3, Package_TO_SOT_SMD:TO-252-3_TabPin2, F.Cu at (71.7, 106.0)
- added R4: 330, Resistor_SMD:R_0805_2012Metric_Pad1.20x1.40mm_HandSolder, F.Cu at (70.3, 111.5)
- added R5: 330, Resistor_SMD:R_0805_2012Metric_Pad1.20x1.40mm_HandSolder, F.Cu at (80.2, 104.8)
- added U2: INA219AxD, Package_SO:SOIC-8_3.9x4.9mm_P1.27mm, F.Cu at (82.0, 97.1)
- added U3: INA181, Package_TO_SOT_SMD:SOT-23-6, F.Cu at (96.1, 106.4)
