File: Source Files/PCB/BBQino/230Vloads.sch (KiCad schematic (older format))
At the start: 31 parts, among them J2 230V input, J3 230V out, K1 FTR-MYAA005D, K2 FTR-MYAA005D, K3 FINDER-40.41, K4 FINDER-40.41, Q6 2N7002K, Q7 2N7002K

Commit message: New architecture
Parts:
- added J4: 230V_1_presence, TerminalBlock_Phoenix:TerminalBlock_Phoenix_PT-1,5-2-3.5-H_1x02_P3.50mm_Horizontal, symbol BBQino-rescue:Screw_Terminal_01x02-Connector
- added J6: 230v_2_presence, TerminalBlock_Phoenix:TerminalBlock_Phoenix_PT-1,5-2-3.5-H_1x02_P3.50mm_Horizontal, symbol BBQino-rescue:Screw_Terminal_01x02-Connector
- D1, D3, D5, D6, D7, D8: symbol Diode:1N4007 -> BBQino-rescue:1N4007-Diode
- D2, D4: symbol Device:LED_ALT -> BBQino-rescue:LED_ALT-Device
- H1, H2: symbol Mechanical:MountingHole -> BBQino-rescue:MountingHole-Mechanical
- J3: symbol Connector:Screw_Terminal_01x04 -> BBQino-rescue:Screw_Terminal_01x04-Connector
- JP1: symbol Jumper:Jumper_2_Open -> BBQino-rescue:Jumper_2_Open-Jumper
- J_K1, J_K11, J_K2, J_K22: symbol Connector:Conn_01x04_Male -> BBQino-rescue:Conn_01x04_Male-Connector
- J_K1_M1, J_K2_M1: symbol Connector:Conn_01x04_Female -> BBQino-rescue:Conn_01x04_Female-Connector
- K3, K4: symbol Relay:FINDER-40.41 -> BBQino-rescue:FINDER-40.41-Relay
- Q6, Q7: symbol Transistor_FET:2N7002K -> BBQino-rescue:2N7002K-Transistor_FET
- R12, R13, R2, R3: symbol Device:R_US -> BBQino-rescue:R_US-Device
Connections:
- wire segments 116 -> 130
Other:
- note added: "230V PRESENCE ext LED\n"
- moved on the sheet: C7, D3, D4, R3
Changed lines of the file:
@@
 $Descr A4 11693 8268
 encoding utf-8
-Sheet 5 6
+Sheet 5 7
 Title ""
 Date ""
@@
 230V_OUT_1
 $Comp
-L Diode:1N4007 D1
+L BBQino-rescue:1N4007-Diode D1
 U 1 1 614D8121
 P 8450 1750
@@
 $EndComp
 $Comp
-L Device:LED_ALT D2
+L BBQino-rescue:LED_ALT-Device D2
 U 1 1 614D944B
 P 9050 1750
@@
 $EndComp
 $Comp
-L Device:R_US R2
+L BBQino-rescue:R_US-Device R2
 U 1 1 614D9B59
 P 8000 2200
@@
 	9050 1900 9050 2200
 Wire Wire Line
-	9050 2200 8450 2200
-Wire Wire Line
 	8450 1900 8450 2200
 Connection ~ 8450 2200
@@
 Wire Notes Line
 	750  3000 750  2200
-Text GLabel 8700 2350 0    50   Input ~ 0
+Text GLabel 8520 2370 0    50   Input ~ 0
 230V_OUT_2
 $Comp
 L BBQino-rescue:ECWFE2J105K C7
 U 1 1 614FFD8B
-P 9300 2350
-F 0 "C7" H 9450 2703 60  0000 C CNN
-F 1 "0.1 uF " H 9450 2597 60  0000 C CNN
-F 2 "BBQino:ECWFE2J105K" H 9450 1990 60  0001 C CNN
-F 3 "" H 9300 2350 60  0001 C CNN
-F 4 "630V" H 9450 2499 50  0000 C CNN "value2"
-	1    9300 2350
-	1    0    0    -1
-$EndComp
-$Comp
-L Device:LED_ALT D4
+P 9120 2370
+F 0 "C7" H 9390 2450 60  0000 C CNN
+F 1 "0.1 uF " H 9300 2150 60  0000 C CNN
+F 2 "BBQino:ECWFE2J105K" H 9270 2010 60  0001 C CNN
+F 3 "" H 9120 2370 60  0001 C CNN
+F 4 "630V" H 9280 2230 50  0000 C CNN "value2"
+	1    9120 2370
+	1    0    0    -1
+$EndComp
+$Comp
+L BBQino-rescue:LED_ALT-Device D4
 U 1 1 614FFD91
-P 10500 2800
-F 0 "D4" V 10539 2682 50  0000 R CNN
-F 1 "LED_ALT" V 10448 2682 50  0000 R CNN
-F 2 "BBQino:150080BS75000" H 10500 2800 50  0001 C CNN
-F 3 "https://www.mouser.it/datasheet/2/445/150080BS75000-1715853.pdf" H 10500 2800 50  0001 C CNN
-	1    10500 2800
+P 10320 2820
+F 0 "D4" V 10359 2702 50  0000 R CNN
+F 1 "LED_ALT" V 10268 2702 50  0000 R CNN
+F 2 "BBQino:150080BS75000" H 10320 2820 50  0001 C CNN
+F 3 "https://www.mouser.it/datasheet/2/445/150080BS75000-1715853.pdf" H 10320 2820 50  0001 C CNN
+	1    10320 2820
 	0    -1   -1   0
 $EndComp
 $Comp
-L Device:R_US R3
+L BBQino-rescue:R_US-Device R3
 U 1 1 614FFD98
-P 9450 3250
-F 0 "R3" V 9155 3250 50  0000 C CNN
-F 1 "22k" V 9246 3250 50  0000 C CNN
-F 2 "Resistor_SMD:R_2010_5025Metric_Pad1.40x2.65mm_HandSolder" V 9490 3240 50  0001 C CNN
-F 3 "~" H 9450 3250 50  0001 C CNN
-F 4 "2W" V 9337 3250 50  0000 C CNN "Value2"
-	1    9450 3250
-	0    1    1    0
-$EndComp
-Wire Wire Line
-	9600 2350 9900 2350
-Wire Wire Line
-	9900 2350 9900 2650
-Wire Wire Line
-	9900 2350 10500 2350
-Wire Wire Line
-	10500 2350 10500 2650
-Connection ~ 9900 2350
-Wire Wire Line
-	10500 2950 10500 3250
-Wire Wire Line
-	10500 3250 9900 3250
-Wire Wire Line
-	9900 2950 9900 3250
-Connection ~ 9900 3250
-Wire Wire Line
-	9900 3250 9600 3250
-Text GLabel 8800 3250 0    50   Input ~ 0
+P 9270 3270
+F 0 "R3" V 8975 3270 50  0000 C CNN
+F 1 "22k" V 9066 3270 50  0000 C CNN
+F 2 "Resistor_SMD:R_2010_5025Metric_Pad1.40x2.65mm_HandSolder" V 9310 3260 50  0001 C CNN
+F 3 "~" H 9270 3270 50  0001 C CNN
+F 4 "2W" V 9157 3270 50  0000 C CNN "Value2"
+	1    9270 3270
+	0    1    1    0
+$EndComp
+Wire Wire Line
+	9420 2370 9720 2370
+Wire Wire Line
+	9720 2370 9720 2670
+Wire Wire Line
+	9720 2370 10120 2370
+Wire Wire Line
+	10320 2370 10320 2670
+Connection ~ 9720 2370
+Wire Wire Line
+	10320 2970 10320 3270
+Wire Wire Line
+	10320 3270 9720 3270
+Wire Wire Line
+	9720 2970 9720 3270
+Connection ~ 9720 3270
+Wire Wire Line
+	9720 3270 9420 3270
+Text GLabel 8620 3270 0    50   Input ~ 0
 230V_N
 Wire Wire Line
-	8800 3250 9300 3250
-Wire Wire Line
-	8700 2350 9300 2350
-$Comp
-L Diode:1N4007 D3
+	8620 3270 9120 3270
+Wire Wire Line
+	8520 2370 9120 2370
+$Comp
+L BBQino-rescue:1N4007-Diode D3
 U 1 1 614FFD84
-P 9900 2800
-F 0 "D3" V 9854 2880 50  0000 L CNN
-F 1 "1N4148W-HF" V 9800 2250 50  0000 L CNN
-F 2 "Diode_SMD:D_SOD-123" H 9900 2625 50  0001 C CNN
-F 3 "https://www.mouser.it/datasheet/2/80/QW-J0017_1N4148W-HF_RevA-1846955.pdf" H 9900 2800 50  0001 C CNN
-	1    9900 2800
+P 9720 2820
+F 0 "D3" V 9674 2900 50  0000 L CNN
+F 1 "1N4148W-HF" V 9730 2260 50  0000 L CNN
+F 2 "Diode_SMD:D_SOD-123" H 9720 2645 50  0001 C CNN
+F 3 "https://www.mouser.it/datasheet/2/80/QW-J0017_1N4148W-HF_RevA-1846955.pdf" H 9720 2820 50  0001 C CNN
+	1    9720 2820
 	0    1    1    0
 $EndComp
@@
 Isolate with potting or conf. coating \nMount these componentes on the bottom. \nProtects against acidental touching
 $Comp
-L Connector:Conn_01x04_Female J_K1_M1
+L BBQino-rescue:Conn_01x04_Female-Connector J_K1_M1
 U 1 1 6151D7D1
 P 4600 2800
@@
 $EndComp
 $Comp
-L Connector:Conn_01x04_Female J_K2_M1
+L BBQino-rescue:Conn_01x04_Female-Connector J_K2_M1
 U 1 1 6151E93A
 P 4600 3450
@@
 	4200 2200 4300 2200
 $Comp
-L Connector:Conn_01x04_Male J_K1
+L BBQino-rescue:Conn_01x04_Male-Connector J_K1
 U 1 1 61525374
 P 2910 4240
@@
 $EndComp
 $Comp
-L Connector:Conn_01x04_Male J_K2
+L BBQino-rescue:Conn_01x04_Male-Connector J_K2
 U 1 1 61527800
 P 2870 4950
@@
 K1
 $Comp
-L Diode:1N4007 D5
+L BBQino-rescue:1N4007-Diode D5
 U 1 1 6157CE68
 P 2200 3800
@@
 $EndComp
 $Comp
-L Diode:1N4007 D6
+L BBQino-rescue:1N4007-Diode D6
 U 1 1 615877B5
 P 2220 4660
@@
 	5035 3350 4800 3350
 $Comp
-L power:GNDD #PWR0114
+L BBQino-rescue:GNDD-power #PWR0114
 U 1 1 615A23E8
 P 5095 3550
@@
 	4800 3550 5095 3550
 $Comp
-L power:GNDD #PWR0115
+L BBQino-rescue:GNDD-power #PWR0115
 U 1 1 615A714B
 P 5095 2900
@@
 230V_N
 $Comp
-L Connector:Screw_Terminal_01x04 J3
+L BBQino-rescue:Screw_Terminal_01x04-Connector J3
 U 1 1 615B8777
 P 5215 4585
@@
 	4949 4785 5015 4785
 $Comp
-L Mechanical:MountingHole H1
+L BBQino-rescue:MountingHole-Mechanical H1
 U 1 1 6151F1F6
 P 10108 5768
@@
 $EndComp
 $Comp
-L Mechanical:MountingHole H2
+L BBQino-rescue:MountingHole-Mechanical H2
 U 1 1 61520C2A
 P 10120 6013
@@
 General purpose 12V relays
 $Comp
-L Diode:1N4007 D7
+L BBQino-rescue:1N4007-Diode D7
 U 1 1 61877E3C
 P 1400 6674
@@
 $EndComp
 $Comp
-L Connector:Conn_01x04_Male J_K11
+L BBQino-rescue:Conn_01x04_Male-Connector J_K11
 U 1 1 61880127
 P 3144 7414
@@
 $EndComp
 $Comp
-L Relay:FINDER-40.41 K3
+L BBQino-rescue:FINDER-40.41-Relay K3
 U 1 1 6188E0AB
 P 2092 6660
@@
 	2292 7146 2404 7146
 $Comp
-L Device:R_US R12
+L BBQino-rescue:R_US-Device R12
 U 1 1 618E9BEB
 P 2570 7314
@@
 	2816 7574 1892 7574
 $Comp
-L power:+12V #PWR0126
+L BBQino-rescue:+12V-power #PWR0126
 U 1 1 619222CD
 P 1892 6112
@@
 $EndComp
 $Comp
-L power:GNDD #PWR0128
+L BBQino-rescue:GNDD-power #PWR0128
 U 1 1 61936220
 P 1202 7358
@@
 $EndComp
 $Comp
-L Jumper:Jumper_2_Open JP1
+L BBQino-rescue:Jumper_2_Open-Jumper JP1
 U 1 1 61939801
 P 986 7220
@@
 	766  7220 766  7368
 $Comp
-L Diode:1N4007 D8
+L BBQino-rescue:1N4007-Diode D8
 U 1 1 61955C23
 P 4110 6630
@@
 $EndComp
 $Comp
-L Connector:Conn_01x04_Male J_K22
+L BBQino-rescue:Conn_01x04_Male-Connector J_K22
 U 1 1 61955C29
 P 5854 7370
@@
 $EndComp
 $Comp
-L Relay:FINDER-40.41 K4
+L BBQino-rescue:FINDER-40.41-Relay K4
 U 1 1 61955C2F
 P 4802 6616
@@
 	5002 7102 5114 7102
 $Comp
-L Device:R_US R13
+L BBQino-rescue:R_US-Device R13
 U 1 1 61955C42
 P 5280 7270
@@
 	4602 7530 4602 7470
 $Comp
-L power:+12V #PWR0129
+L BBQino-rescue:+12V-power #PWR0129
 U 1 1 61955C55
 P 4602 6068
@@
 	1892 7574 1892 7514
 $Comp
-L Transistor_FET:2N7002K Q6
+L BBQino-rescue:2N7002K-Transistor_FET Q6
 U 1 1 619816C3
 P 1992 7314
@@
 $EndComp
 $Comp
-L Transistor_FET:2N7002K Q7
+L BBQino-rescue:2N7002K-Transistor_FET Q7
 U 1 1 619A122F
 P 4702 7270
@@
 	-1   0    0    -1
 $EndComp
+$Comp
+L BBQino-rescue:Screw_Terminal_01x02-Connector J6
+U 1 1 61AC8591
+P 10470 1940
+F 0 "J6" H 10550 1886 50  0000 L CNN
+F 1 "230v_2_presence" H 10550 1841 50  0001 L CNN
+F 2 "TerminalBlock_Phoenix:TerminalBlock_Phoenix_PT-1,5-2-3.5-H_1x02_P3.50mm_Horizontal" H 10470 1940 50  0001 C CNN
+F 3 "" H 10470 1940 50  0001 C CNN
+	1    10470 1940
+	1    0    0    -1
+$EndComp
+$Comp
+L BBQino-rescue:Screw_Terminal_01x02-Connector J4
+U 1 1 61AC9326
+P 10470 1610
+F 0 "J4" H 10550 1556 50  0000 L CNN
+F 1 "230V_1_presence" H 10550 1511 50  0001 L CNN
+F 2 "TerminalBlock_Phoenix:TerminalBlock_Phoenix_PT-1,5-2-3.5-H_1x02_P3.50mm_Horizontal" H 10470 1610 50  0001 C CNN
+F 3 "" H 10470 1610 50  0001 C CNN
+	1    10470 1610
+	1    0    0    -1
+$EndComp
+Text Notes 9940 1460 0    50   ~ 0
+230V PRESENCE ext LED\n
+Wire Notes Line
+	9910 1420 9870 1420
+Wire Notes Line
+	9870 1420 9870 2210
+Wire Notes Line
+	9870 2210 10960 2210
+Wire Wire Line
+	9050 1300 9700 1300
+Wire Wire Line
+	9700 1300 9700 1610
+Wire Wire Line
+	9700 1610 10270 1610
+Connection ~ 9050 1300
+Wire Wire Line
+	10270 1710 9700 1710
+Wire Wire Line
+	9700 1710 9700 2200
+Wire Wire Line
+	8450 2200 9050 2200
+Connection ~ 9050 2200
+Wire Wire Line
+	9050 2200 9700 2200
+Wire Wire Line
+	10270 2040 10270 2280
+Wire Wire Line
+	10270 2280 10860 2280
+Wire Wire Line
+	10860 2280 10860 3270
+Wire Wire Line
+	10860 3270 10320 3270
+Connection ~ 10320 3270
+Wire Wire Line
+	9720 2370 10120 2370
+Wire Wire Line
+	10120 2370 10120 1940
+Wire Wire Line
+	10120 1940 10270 1940
+Connection ~ 10120 2370
+Wire Wire Line
+	10120 2370 10320 2370
 $EndSCHEMATC
