File: Source Files/PCB/BBQino/Thermocouple.sch (KiCad schematic (older format))
At the start: 5 parts

Commit message: added current sense on motor side
Parts:
- gave numbers to parts that had none: 5
Changed lines of the file:
@@
 MAX6675\nType -K Thermocouple\n\n● Cold-Junction Compensation\n● Simple SPI-Compatible Serial Interface\n● 12-Bit, 0.25°C Resolution\n● Open Thermocouple Detection
 $Comp
-L BBQino-rescue:MAX6675ISA+T IC?
+L BBQino-rescue:MAX6675ISA+T IC3
 U 1 1 615ACA16
 P 3970 3575
-F 0 "IC?" H 4520 3840 50  0000 C CNN
+F 0 "IC3" H 4520 3840 50  0000 C CNN
 F 1 "MAX6675ISA+T" H 4520 3749 50  0000 C CNN
 F 2 "BBQino:SOIC127P600X175-8N" H 4920 3675 50  0001 L CNN
@@
 $EndComp
 $Comp
-L BBQino-rescue:DG4052EEN-T1-GE4 IC?
+L BBQino-rescue:DG4052EEN-T1-GE4 IC2
 U 1 1 615ADDB4
 P 2145 3750
-F 0 "IC?" H 3105 3020 50  0000 L CNN
+F 0 "IC2" H 3105 3020 50  0000 L CNN
 F 1 "DG4052EEN-T1-GE4" H 3105 2933 50  0000 L CNN
 F 2 "BBQino:QFN40P180X260X60-16N-D" H 3095 4050 50  0001 L CNN
@@
 $EndComp
 $Comp
-L Device:Thermocouple TC?
+L Device:Thermocouple TC1
 U 1 1 615AEE20
 P 1405 3505
-F 0 "TC?" H 1378 3830 50  0000 C CNN
+F 0 "TC1" H 1378 3830 50  0000 C CNN
 F 1 "Thermocouple" H 1378 3739 50  0000 C CNN
 F 2 "" H 830 3555 50  0001 C CNN
@@
 $EndComp
 $Comp
-L Device:Thermocouple TC?
+L Device:Thermocouple TC2
 U 1 1 615AF447
 P 1435 4245
-F 0 "TC?" H 1408 4570 50  0000 C CNN
+F 0 "TC2" H 1408 4570 50  0000 C CNN
 F 1 "Thermocouple" H 1408 4479 50  0000 C CNN
 F 2 "" H 860 4295 50  0001 C CNN
@@
 $EndComp
 $Comp
-L Device:Thermocouple TC?
+L Device:Thermocouple TC3
 U 1 1 615AF6AE
 P 1435 5095
-F 0 "TC?" H 1408 5420 50  0000 C CNN
+F 0 "TC3" H 1408 5420 50  0000 C CNN
 F 1 "Thermocouple" H 1408 5329 50  0000 C CNN
 F 2 "" H 860 5145 50  0001 C CNN
@@
 	2695 3195 2695 3250
 $Comp
-L power:+5VA #PWR?
+L power:+5VA #PWR0122
 U 1 1 615BEA1C
 P 2795 3140
-F 0 "#PWR?" H 2795 2990 50  0001 C CNN
+F 0 "#PWR0122" H 2795 2990 50  0001 C CNN
 F 1 "+5VA" H 2810 3313 50  0000 C CNN
 F 2 "" H 2795 3140 50  0001 C CNN
@@
 	2795 3250 2795 3140
 $Comp
-L power:GNDA #PWR?
+L power:GNDA #PWR0123
 U 1 1 615C0417
 P 2595 4880
-F 0 "#PWR?" H 2595 4630 50  0001 C CNN
+F 0 "#PWR0123" H 2595 4630 50  0001 C CNN
 F 1 "GNDA" H 2600 4707 50  0000 C CNN
 F 2 "" H 2595 4880 50  0001 C CNN
@@
 	3280 3750 3245 3750
 $Comp
-L power:+5VA #PWR?
+L power:+5VA #PWR0124
 U 1 1 615DC0DB
 P 3970 3875
-F 0 "#PWR?" H 3970 3725 50  0001 C CNN
+F 0 "#PWR0124" H 3970 3725 50  0001 C CNN
 F 1 "+5VA" H 3985 4048 50  0000 C CNN
 F 2 "" H 3970 3875 50  0001 C CNN
@@
 $EndComp
 $Comp
-L power:GNDA #PWR?
+L power:GNDA #PWR0125
 U 1 1 615DC6B6
 P 3970 3575
-F 0 "#PWR?" H 3970 3325 50  0001 C CNN
+F 0 "#PWR0125" H 3970 3325 50  0001 C CNN
 F 1 "GNDA" H 3975 3402 50  0000 C CNN
 F 2 "" H 3970 3575 50  0001 C CNN

Commit message: New architecture
Parts:
- TC1, TC2, TC3: symbol Device:Thermocouple -> BBQino-rescue:Thermocouple-Device
Changed lines of the file:
@@
 $Descr A4 11693 8268
 encoding utf-8
-Sheet 6 6
+Sheet 6 7
 Title ""
 Date ""
@@
 $EndComp
 $Comp
-L Device:Thermocouple TC1
+L BBQino-rescue:Thermocouple-Device TC1
 U 1 1 615AEE20
 P 1405 3505
@@
 $EndComp
 $Comp
-L Device:Thermocouple TC2
+L BBQino-rescue:Thermocouple-Device TC2
 U 1 1 615AF447
 P 1435 4245
@@
 $EndComp
 $Comp
-L Device:Thermocouple TC3
+L BBQino-rescue:Thermocouple-Device TC3
 U 1 1 615AF6AE
 P 1435 5095
@@
 	2695 3195 2695 3250
 $Comp
-L power:+5VA #PWR0122
+L BBQino-rescue:+5VA-power #PWR0122
 U 1 1 615BEA1C
 P 2795 3140
@@
 	2795 3250 2795 3140
 $Comp
-L power:GNDA #PWR0123
+L BBQino-rescue:GNDA-power #PWR0123
 U 1 1 615C0417
 P 2595 4880
@@
 	3280 3750 3245 3750
 $Comp
-L power:+5VA #PWR0124
+L BBQino-rescue:+5VA-power #PWR0124
 U 1 1 615DC0DB
 P 3970 3875
@@
 $EndComp
 $Comp
-L power:GNDA #PWR0125
+L BBQino-rescue:GNDA-power #PWR0125
 U 1 1 615DC6B6
 P 3970 3575
